File: sendit/sendit.kicad_pcb (KiCad board)
At the start: 2 copper layers, 33 parts, among them U1 ADS1115IDGS, U2 Seeed_Studio_XIAO_ESP32C6, U3 ADS1115IDGS

Commit message: big update on the potential design.
Parts:
- added C10: 100nF, Capacitor_SMD:C_0805_2012Metric_Pad1.18x1.45mm_HandSolder, F.Cu at (144.6, 127.5)
- added C11: 100nF, Capacitor_SMD:C_0805_2012Metric_Pad1.18x1.45mm_HandSolder, F.Cu at (91.5, 137.9)
- added C12: 100nF, Capacitor_SMD:C_0805_2012Metric_Pad1.18x1.45mm_HandSolder, F.Cu at (155.8, 115.2)
- added C13: 100nF, Capacitor_SMD:C_0805_2012Metric_Pad1.18x1.45mm_HandSolder, F.Cu at (144.6, 68.6)
- added C14: 100nF, Capacitor_SMD:C_0805_2012Metric_Pad1.18x1.45mm_HandSolder, F.Cu at (166.9, 115.2)
- added C15: 100nF, Capacitor_SMD:C_0805_2012Metric_Pad1.18x1.45mm_HandSolder, F.Cu at (121.4, 68.6)
- added C16: 100nF, Capacitor_SMD:C_0805_2012Metric_Pad1.18x1.45mm_HandSolder, F.Cu at (144.6, 115.2)
- added C17: 100nF, Capacitor_SMD:C_0805_2012Metric_Pad1.18x1.45mm_HandSolder, F.Cu at (121.4, 103.0)
- added C18: 100nF, Capacitor_SMD:C_0805_2012Metric_Pad1.18x1.45mm_HandSolder, F.Cu at (166.9, 127.5)
- added C19: 100nF, Capacitor_SMD:C_0805_2012Metric_Pad1.18x1.45mm_HandSolder, F.Cu at (144.6, 103.0)
- added C20: 100nF, Capacitor_SMD:C_0805_2012Metric_Pad1.18x1.45mm_HandSolder, F.Cu at (155.8, 127.5)
- added C21: 10uF, Capacitor_SMD:C_0805_2012Metric_Pad1.18x1.45mm_HandSolder, F.Cu at (65.3, 57.7)
- added C5: 100nF, Capacitor_SMD:C_0805_2012Metric_Pad1.18x1.45mm_HandSolder, F.Cu at (155.8, 139.7)
- added C6: 100nF, Capacitor_SMD:C_0805_2012Metric_Pad1.18x1.45mm_HandSolder, F.Cu at (121.4, 120.2)
- added C7: 100nF, Capacitor_SMD:C_0805_2012Metric_Pad1.18x1.45mm_HandSolder, F.Cu at (132.9, 129.8)
- added C8: 10uF, Capacitor_SMD:C_0805_2012Metric_Pad1.18x1.45mm_HandSolder, F.Cu at (132.9, 132.9)
- added C9: 100nF, Capacitor_SMD:C_0805_2012Metric_Pad1.18x1.45mm_HandSolder, F.Cu at (144.6, 139.7)
- added J1: ~, Connector_PinHeader_2.54mm:PinHeader_2x03_P2.54mm_Vertical, F.Cu at (158.6, 74.5)
- added J2: ~, Connector_PinHeader_2.54mm:PinHeader_2x03_P2.54mm_Vertical, F.Cu at (135.3, 74.5)
- added J3: ~, Connector_PinHeader_2.54mm:PinHeader_2x03_P2.54mm_Vertical, F.Cu at (135.3, 108.8)
- added J4: ~, Connector_PinHeader_2.54mm:PinHeader_2x03_P2.54mm_Vertical, F.Cu at (105.5, 126.5)
- added J5: ~, Connector_PinHeader_2.54mm:PinHeader_2x03_P2.54mm_Vertical, F.Cu at (158.6, 57.3)
- added J6: ~, Connector_PinHeader_2.54mm:PinHeader_2x03_P2.54mm_Vertical, F.Cu at (135.3, 57.3)
- added J7: ~, Connector_PinHeader_2.54mm:PinHeader_2x03_P2.54mm_Vertical, F.Cu at (135.3, 91.6)
- added J8: ~, Connector_PinHeader_2.54mm:PinHeader_2x03_P2.54mm_Vertical, F.Cu at (158.6, 91.6)
- added J9: Micro_SD_Card, Connector_Card:microSD_HC_Hirose_DM3AT-SF-PEJM5, F.Cu at (54.5, 65.5)
- added R11: 1k, Resistor_SMD:R_0805_2012Metric_Pad1.20x1.40mm_HandSolder, F.Cu at (126.2, 120.2)
- added R12: 10k, Resistor_SMD:R_0805_2012Metric_Pad1.20x1.40mm_HandSolder, F.Cu at (137.7, 129.8)
- added R13: 165 0.1%, Resistor_SMD:R_1206_3216Metric_Pad1.30x1.75mm_HandSolder, F.Cu at (176.4, 56.6)
- added R14: 13K 0.1%, Resistor_SMD:R_1206_3216Metric_Pad1.30x1.75mm_HandSolder, F.Cu at (168.5, 99.5)
- added R15: 1.5K 0.1%, Resistor_SMD:R_1206_3216Metric_Pad1.30x1.75mm_HandSolder, F.Cu at (168.5, 102.8)
- added R16: 910 0.1%, Resistor_SMD:R_1206_3216Metric_Pad1.30x1.75mm_HandSolder, F.Cu at (80.6, 78.3)
- added R17: 1k 0.1%, Resistor_SMD:R_1206_3216Metric_Pad1.30x1.75mm_HandSolder, F.Cu at (73.0, 86.4)
- added R18: 165 0.1%, Resistor_SMD:R_1206_3216Metric_Pad1.30x1.75mm_HandSolder, F.Cu at (145.2, 144.9)
- added R19: 1k, Resistor_SMD:R_0805_2012Metric_Pad1.20x1.40mm_HandSolder, F.Cu at (96.3, 137.8)
- added R20: 13K 0.1%, Resistor_SMD:R_1206_3216Metric_Pad1.30x1.75mm_HandSolder, F.Cu at (176.4, 82.3)
- added R21: 1.5K 0.1%, Resistor_SMD:R_1206_3216Metric_Pad1.30x1.75mm_HandSolder, F.Cu at (176.4, 85.6)
- added R22: 165 0.1%, Resistor_SMD:R_1206_3216Metric_Pad1.30x1.75mm_HandSolder, F.Cu at (108.0, 143.0)
- added R23: 470 0.1%, Resistor_SMD:R_1206_3216Metric_Pad1.30x1.75mm_HandSolder, F.Cu at (80.6, 66.4)
- added R24: 1k 0.1%, Resistor_SMD:R_1206_3216Metric_Pad1.30x1.75mm_HandSolder, F.Cu at (65.0, 91.7)
- added R25: 1k, Resistor_SMD:R_0805_2012Metric_Pad1.20x1.40mm_HandSolder, F.Cu at (149.4, 68.6)
- added R26: 910 0.1%, Resistor_SMD:R_1206_3216Metric_Pad1.30x1.75mm_HandSolder, F.Cu at (80.6, 69.7)
- added R27: 1k 0.1%, Resistor_SMD:R_1206_3216Metric_Pad1.30x1.75mm_HandSolder, F.Cu at (57.0, 91.7)
- added R28: 13K 0.1%, Resistor_SMD:R_1206_3216Metric_Pad1.30x1.75mm_HandSolder, F.Cu at (168.5, 82.3)
- added R29: 1.5K 0.1%, Resistor_SMD:R_1206_3216Metric_Pad1.30x1.75mm_HandSolder, F.Cu at (168.5, 85.6)
- added R30: 165 0.1%, Resistor_SMD:R_1206_3216Metric_Pad1.30x1.75mm_HandSolder, F.Cu at (92.1, 143.0)
- added R31: 470 0.1%, Resistor_SMD:R_1206_3216Metric_Pad1.30x1.75mm_HandSolder, F.Cu at (72.7, 57.8)
- added R32: 1k 0.1%, Resistor_SMD:R_1206_3216Metric_Pad1.30x1.75mm_HandSolder, F.Cu at (73.0, 91.7)
- added R33: 1k, Resistor_SMD:R_0805_2012Metric_Pad1.20x1.40mm_HandSolder, F.Cu at (126.2, 68.6)
- added R34: 13K 0.1%, Resistor_SMD:R_1206_3216Metric_Pad1.30x1.75mm_HandSolder, F.Cu at (168.5, 56.6)
- added R35: 1.5K 0.1%, Resistor_SMD:R_1206_3216Metric_Pad1.30x1.75mm_HandSolder, F.Cu at (168.5, 59.9)
- added R36: 165 0.1%, Resistor_SMD:R_1206_3216Metric_Pad1.30x1.75mm_HandSolder, F.Cu at (100.0, 143.0)
- added R37: 910 0.1%, Resistor_SMD:R_1206_3216Metric_Pad1.30x1.75mm_HandSolder, F.Cu at (72.7, 61.1)
- added R38: 1k 0.1%, Resistor_SMD:R_1206_3216Metric_Pad1.30x1.75mm_HandSolder, F.Cu at (57.0, 97.0)
- added R39: 1k, Resistor_SMD:R_0805_2012Metric_Pad1.20x1.40mm_HandSolder, F.Cu at (126.2, 103.0)
- added R40: 13K 0.1%, Resistor_SMD:R_1206_3216Metric_Pad1.30x1.75mm_HandSolder, F.Cu at (175.4, 141.2)
- added R41: 1.5K 0.1%, Resistor_SMD:R_1206_3216Metric_Pad1.30x1.75mm_HandSolder, F.Cu at (175.4, 144.5)
- added R42: 165 0.1%, Resistor_SMD:R_1206_3216Metric_Pad1.30x1.75mm_HandSolder, F.Cu at (176.4, 67.2)
- added R43: 470 0.1%, Resistor_SMD:R_1206_3216Metric_Pad1.30x1.75mm_HandSolder, F.Cu at (80.6, 57.8)
- added R44: 1k 0.1%, Resistor_SMD:R_1206_3216Metric_Pad1.30x1.75mm_HandSolder, F.Cu at (73.0, 97.0)
- added R45: 1k, Resistor_SMD:R_0805_2012Metric_Pad1.20x1.40mm_HandSolder, F.Cu at (149.4, 103.0)
- added R46: 13K 0.1%, Resistor_SMD:R_1206_3216Metric_Pad1.30x1.75mm_HandSolder, F.Cu at (121.9, 138.0)
- added R47: 1.5K 0.1%, Resistor_SMD:R_1206_3216Metric_Pad1.30x1.75mm_HandSolder, F.Cu at (121.9, 141.3)
- added R48: 165 0.1%, Resistor_SMD:R_1206_3216Metric_Pad1.30x1.75mm_HandSolder, F.Cu at (176.4, 61.9)
- added R49: 910 0.1%, Resistor_SMD:R_1206_3216Metric_Pad1.30x1.75mm_HandSolder, F.Cu at (80.6, 61.1)
- added R50: 1k 0.1%, Resistor_SMD:R_1206_3216Metric_Pad1.30x1.75mm_HandSolder, F.Cu at (65.0, 86.4)
- added R51: 1k 0.1%, Resistor_SMD:R_1206_3216Metric_Pad1.30x1.75mm_HandSolder, F.Cu at (65.0, 97.0)
- added R52: 470 0.1%, Resistor_SMD:R_1206_3216Metric_Pad1.30x1.75mm_HandSolder, F.Cu at (49.1, 86.4)
- added R53: 910 0.1%, Resistor_SMD:R_1206_3216Metric_Pad1.30x1.75mm_HandSolder, F.Cu at (49.1, 89.7)
- added R54: 470 0.1%, Resistor_SMD:R_1206_3216Metric_Pad1.30x1.75mm_HandSolder, F.Cu at (49.1, 95.0)
- added R55: 910 0.1%, Resistor_SMD:R_1206_3216Metric_Pad1.30x1.75mm_HandSolder, F.Cu at (49.1, 98.3)
- added R56: 470 0.1%, Resistor_SMD:R_1206_3216Metric_Pad1.30x1.75mm_HandSolder, F.Cu at (72.7, 66.4)
- added R57: 910 0.1%, Resistor_SMD:R_1206_3216Metric_Pad1.30x1.75mm_HandSolder, F.Cu at (72.7, 69.7)
- added R58: 470 0.1%, Resistor_SMD:R_1206_3216Metric_Pad1.30x1.75mm_HandSolder, F.Cu at (72.7, 75.0)
- added R59: 910 0.1%, Resistor_SMD:R_1206_3216Metric_Pad1.30x1.75mm_HandSolder, F.Cu at (72.7, 78.3)
- added R60: 10k, Resistor_SMD:R_0805_2012Metric_Pad1.20x1.40mm_HandSolder, F.Cu at (65.2, 60.6)
- added R61: 4.7k, Resistor_SMD:R_0805_2012Metric_Pad1.20x1.40mm_HandSolder, F.Cu at (65.2, 63.6)
- added R62: 4.7k, Resistor_SMD:R_0805_2012Metric_Pad1.20x1.40mm_HandSolder, F.Cu at (65.2, 66.5)
- added R63: 4.7k, Resistor_SMD:R_0805_2012Metric_Pad1.20x1.40mm_HandSolder, F.Cu at (65.2, 69.5)
- added R64: 220, Resistor_SMD:R_0805_2012Metric_Pad1.20x1.40mm_HandSolder, F.Cu at (65.2, 72.5)
- added R65: 220, Resistor_SMD:R_0805_2012Metric_Pad1.20x1.40mm_HandSolder, F.Cu at (65.2, 75.4)
- added R66: 220, Resistor_SMD:R_0805_2012Metric_Pad1.20x1.40mm_HandSolder, F.Cu at (65.2, 78.3)
- added R67: 10k, Resistor_SMD:R_0805_2012Metric_Pad1.20x1.40mm_HandSolder, F.Cu at (65.2, 81.3)
- added U10: TMUX4052PWR, yarrboard:TSSOP16-PW_TEX, F.Cu at (146.7, 110.4)
- added U11: TMUX4052PWR, yarrboard:TSSOP16-PW_TEX, F.Cu at (169.0, 122.6)
- added U12: TMUX4052PWR, yarrboard:TSSOP16-PW_TEX, F.Cu at (157.9, 122.6)
- added U4: ADS1115IDGS, Package_SO:TSSOP-10_3x3mm_P0.5mm, F.Cu at (134.0, 126.0)
- added U5: TMUX4052PWR, yarrboard:TSSOP16-PW_TEX, F.Cu at (146.7, 134.8)
- added U6: TMUX4052PWR, yarrboard:TSSOP16-PW_TEX, F.Cu at (146.7, 122.6)
- added U7: TMUX4052PWR, yarrboard:TSSOP16-PW_TEX, F.Cu at (157.9, 110.4)
- added U8: TMUX4052PWR, yarrboard:TSSOP16-PW_TEX, F.Cu at (169.0, 110.4)
- added U9: TPS61040DBV, Package_TO_SOT_SMD:SOT-23-5, F.Cu at (137.4, 138.8)
- C2, C4: value 10uF -> 100nF
- C3: value 100nF -> 10uF
- D1, D2, D3, D4, D5, D6, D7, D8: value BAT54S -> BAV199
- R1, R7: value 249 0.1% -> 1k; footprint Resistor_SMD:R_1206_3216Metric_Pad1.30x1.75mm_HandSolder -> Resistor_SMD:R_0805_2012Metric_Pad1.20x1.40mm_HandSolder
- R10: value 10k -> 1.5K 0.1%; footprint Resistor_SMD:R_0805_2012Metric_Pad1.20x1.40mm_HandSolder -> Resistor_SMD:R_1206_3216Metric_Pad1.30x1.75mm_HandSolder
- R2: value 10k -> 470 0.1%; footprint Resistor_SMD:R_0805_2012Metric_Pad1.20x1.40mm_HandSolder -> Resistor_SMD:R_1206_3216Metric_Pad1.30x1.75mm_HandSolder
- R3: value 249 0.1% -> 10K
- R4, R9: value 249 0.1% -> 13K 0.1%
- R5: value 249 0.1% -> 1.5K 0.1%
- R6: value 249 0.1% -> 10k; footprint Resistor_SMD:R_1206_3216Metric_Pad1.30x1.75mm_HandSolder -> Resistor_SMD:R_0805_2012Metric_Pad1.20x1.40mm_HandSolder
- R8: value 249 0.1% -> 165 0.1%
- U1: value ADS1115IDGS -> ~; footprint Package_SO:TSSOP-10_3x3mm_P0.5mm -> yarrboard:Waveshare-ESP32-S3-dev-kit-SMD
- U2: value Seeed_Studio_XIAO_ESP32C6 -> ADS1115IDGS; footprint Seeed Studio XIAO Series Library:XIAO-Generic-Hybrid-14P-2.54-21X17.8MM -> Package_SO:TSSOP-10_3x3mm_P0.5mm
- U3: value ADS1115IDGS -> TMUX4052PWR; footprint Package_SO:TSSOP-10_3x3mm_P0.5mm -> yarrboard:TSSOP16-PW_TEX
- moved R10 199.1 mm to (175.4, 135.9)
- moved U3 187.3 mm to (157.9, 134.8)
- moved C3 152.7 mm to (121.4, 132.9)
- moved C1 149.7 mm to (144.6, 85.8)
- moved R9 148.6 mm to (175.4, 132.6)
- moved R5 146.9 mm to (176.4, 94.2)
- moved R4 145.8 mm to (176.4, 91.0)
- moved R8 145.5 mm to (156.3, 144.9)
- moved C2 139.7 mm to (121.4, 129.8)
- moved C4 137.6 mm to (121.4, 85.8)
- moved U2 118.1 mm to (122.4, 126.0)
- moved D5 116.1 mm to (158.7, 67.0)
- moved D7 116.1 mm to (135.5, 101.4)
- moved D2 116.0 mm to (135.5, 84.2)
- moved D8 115.5 mm to (158.7, 101.4)
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Connections:
- C1 pad 1: +5V -> /ADC1/ADC0
- C1 pad 2: GNDA -> GND
- C2 pad 1: +5V -> +3.3V
- C2 pad 2: GNDA -> GND
- C3 pad 1: +5V -> +3.3V
- C3 pad 2: GNDA -> GND
- C4 pad 1: +5V -> /ADC2/ADC0
- C4 pad 2: GNDA -> GND
- D1 pad 2: +5V -> +3.3V
- D2 pad 2: +5V -> +3.3V
- D2 pad 3: /ADC1/ADC1 -> /ADC2/ADC0
- D3 pad 2: +5V -> +3.3V
- D3 pad 3: /ADC1/ADC2 -> /ADC1/ADC1
- D4 pad 2: +5V -> +3.3V
- D4 pad 3: /ADC1/ADC3 -> /ADC1/ADC2
- D5 pad 2: +5V -> +3.3V
- D5 pad 3: /ADC2/ADC0 -> /ADC1/ADC3
- D6 pad 2: +5V -> +3.3V
- D7 pad 2: +5V -> +3.3V
- D8 pad 2: +5V -> +3.3V
- INPUT1 pad 1: +5V -> Net-(INPUT1-Pin_1)
- INPUT1 pad 2: /ADC1/ADC0 -> /Analog Channel 1/ADC MUX - TMUX4052/DA
- INPUT2 pad 1: +5V -> Net-(INPUT2-Pin_1)
- INPUT2 pad 2: /ADC1/ADC1 -> /Analog Channel 5/ADC MUX - TMUX4052/DA
- INPUT3 pad 1: +5V -> Net-(INPUT3-Pin_1)
- INPUT3 pad 2: /ADC1/ADC2 -> /Analog Channel 2/ADC MUX - TMUX4052/DA
- INPUT4 pad 1: +5V -> Net-(INPUT4-Pin_1)
- INPUT4 pad 2: /ADC1/ADC3 -> /Analog Channel 3/ADC MUX - TMUX4052/DA
- INPUT5 pad 1: +5V -> Net-(INPUT5-Pin_1)
- INPUT5 pad 2: /ADC2/ADC0 -> /Analog Channel 4/ADC MUX - TMUX4052/DA
- INPUT6 pad 1: +5V -> Net-(INPUT6-Pin_1)
- INPUT6 pad 2: /ADC2/ADC1 -> /Analog Channel 6/ADC MUX - TMUX4052/DA
- INPUT7 pad 1: +5V -> Net-(INPUT7-Pin_1)
- INPUT7 pad 2: /ADC2/ADC2 -> /Analog Channel 7/ADC MUX - TMUX4052/DA
- INPUT8 pad 1: +5V -> Net-(INPUT8-Pin_1)
- INPUT8 pad 2: /ADC2/ADC3 -> /Analog Channel 8/ADC MUX - TMUX4052/DA
- R1 pad 1: GND -> /Analog Channel 1/ADC MUX - TMUX4052/DB
- R10 pad 1: Net-(U3-ALERT/RDY) -> GND
- R10 pad 2: +5V -> /Analog Channel 2/0-32v/OUTPUT
- R2 pad 1: Net-(U1-ALERT/RDY) -> /Analog Channel 1/0-5v/OUTPUT
- R2 pad 2: +5V -> /Analog Channel 1/0-5v/INPUT
- R3 pad 1: GND -> MUX_ENABLE
- R3 pad 2: /ADC1/ADC1 -> +3.3V
- R4 pad 1: GND -> /Analog Channel 1/0-32v/OUTPUT
- R4 pad 2: /ADC1/ADC2 -> /Analog Channel 1/0-32v/INPUT
- R5 pad 2: /ADC1/ADC3 -> /Analog Channel 1/0-32v/OUTPUT
- R6 pad 1: GND -> Net-(U2-ALERT/RDY)
- R6 pad 2: /ADC2/ADC0 -> +3.3V
- R7 pad 1: GND -> /Analog Channel 5/ADC MUX - TMUX4052/DB
- R7 pad 2: /ADC2/ADC1 -> /ADC2/ADC0
- R8 pad 2: /ADC2/ADC2 -> /Analog Channel 1/4-20mA/INPUT
- R9 pad 1: GND -> /Analog Channel 2/0-32v/OUTPUT
- R9 pad 2: /ADC2/ADC3 -> /Analog Channel 2/0-32v/INPUT
- U1 pad 1: +5V -> +3.3V
- U1 pad 10: SCL -> CH6_A0
- U1 pad 2: Net-(U1-ALERT/RDY) -> +3.3V
- U1 pad 3: GNDA -> unconnected-(U1-RST-Pad3)
- U1 pad 4: /ADC1/ADC0 -> unconnected-(U1-GPIO4-Pad4)
- U1 pad 5: /ADC1/ADC1 -> CH8_A1
- U1 pad 6: /ADC1/ADC2 -> CH8_A0
- U1 pad 7: /ADC1/ADC3 -> CH7_A1
- U1 pad 8: +5V -> CH7_A0
- U1 pad 9: SDA -> CH6_A1
- U2 pad 1: unconnected-(U2-D0-Pad1) -> +3.3V
- U2 pad 10: unconnected-(U2-D9-Pad10) -> SCL
- U2 pad 2: unconnected-(U2-D1-Pad2) -> Net-(U2-ALERT/RDY)
- U2 pad 3: unconnected-(U2-D2-Pad3) -> GND
- U2 pad 4: unconnected-(U2-D3-Pad4) -> /ADC2/ADC0
- U2 pad 5: SDA -> /ADC2/ADC1
- U2 pad 6: SCL -> /ADC2/ADC2
- U2 pad 7: unconnected-(U2-D6-Pad7) -> /ADC2/ADC3
- U2 pad 8: unconnected-(U2-D7-Pad8) -> +3.3V
- U2 pad 9: unconnected-(U2-D8-Pad9) -> SDA
- U3 pad 1: GND -> /Analog Channel 2/4-20mA/INPUT
- U3 pad 10: SCL -> CH1_A0
- U3 pad 2: Net-(U3-ALERT/RDY) -> /Analog Channel 2/0-1000 ohm/INPUT
- U3 pad 3: GNDA -> /Analog Channel 2/ADC MUX - TMUX4052/DB
- U3 pad 4: /ADC2/ADC0 -> /Analog Channel 2/0-5v/OUTPUT
- U3 pad 5: /ADC2/ADC1 -> /Analog Channel 2/0-32v/OUTPUT
- U3 pad 6: /ADC2/ADC2 -> MUX_ENABLE
- U3 pad 7: /ADC2/ADC3 -> GND
- U3 pad 8: +5V -> GND
- U3 pad 9: SDA -> CH1_A1

Commit message: bigger update
Parts:
- removed R38, R44, R50, R51: 1k 0.1%, Resistor_SMD:R_1206_3216Metric_Pad1.30x1.75mm_HandSolder
- removed R43, R52, R54, R56, R58: 470 0.1%, Resistor_SMD:R_1206_3216Metric_Pad1.30x1.75mm_HandSolder
- removed R46: 13K 0.1%, Resistor_SMD:R_1206_3216Metric_Pad1.30x1.75mm_HandSolder
- removed R47: 1.5K 0.1%, Resistor_SMD:R_1206_3216Metric_Pad1.30x1.75mm_HandSolder
- removed R49, R53, R55, R57, R59: 910 0.1%, Resistor_SMD:R_1206_3216Metric_Pad1.30x1.75mm_HandSolder
- removed U10, U11, U12, U3, U5, U6, U7, U8: TMUX4052PWR, yarrboard:TSSOP16-PW_TEX
- added D10: BAV199, Package_TO_SOT_SMD:SOT-23, F.Cu at (87.0, 109.0)
- added D11: BAV199, Package_TO_SOT_SMD:SOT-23, F.Cu at (102.0, 109.0)
- added D12: BAV199, Package_TO_SOT_SMD:SOT-23, F.Cu at (117.0, 109.0)
- added D13: BAV199, Package_TO_SOT_SMD:SOT-23, F.Cu at (153.7, 156.1)
- added D14: BAV199, Package_TO_SOT_SMD:SOT-23, F.Cu at (144.6, 156.1)
- added D15: BAV199, Package_TO_SOT_SMD:SOT-23, F.Cu at (132.0, 109.0)
- added D16: BAV199, Package_TO_SOT_SMD:SOT-23, F.Cu at (153.7, 169.2)
- added D17: MBR0530, Diode_SMD:D_SOD-123, F.Cu at (102.0, 165.0)
- added D9: BAV199, Package_TO_SOT_SMD:SOT-23, F.Cu at (72.0, 109.5)
- added F1: 30v / 30mA, Fuse:Fuse_0603_1608Metric, F.Cu at (66.5, 109.0)
- added F2: 30v / 30mA, Fuse:Fuse_0603_1608Metric, F.Cu at (81.5, 108.5)
- added F3: 30v / 30mA, Fuse:Fuse_0603_1608Metric, F.Cu at (96.5, 108.5)
- added F4: 30v / 30mA, Fuse:Fuse_0603_1608Metric, F.Cu at (111.5, 108.5)
- added F5: 30v / 30mA, Fuse:Fuse_0603_1608Metric, F.Cu at (148.2, 155.6)
- added F6: 30v / 30mA, Fuse:Fuse_0603_1608Metric, F.Cu at (139.1, 155.6)
- added F7: 30v / 30mA, Fuse:Fuse_0603_1608Metric, F.Cu at (126.5, 108.5)
- added F8: 30v / 30mA, Fuse:Fuse_0603_1608Metric, F.Cu at (148.2, 168.7)
- added R70: 165 0.1%, Resistor_SMD:R_1206_3216Metric_Pad1.30x1.75mm_HandSolder, F.Cu at (107.0, 37.3)
- added R71: 165 0.1%, Resistor_SMD:R_1206_3216Metric_Pad1.30x1.75mm_HandSolder, F.Cu at (68.7, 59.0)
- added R72: 165 0.1%, Resistor_SMD:R_1206_3216Metric_Pad1.30x1.75mm_HandSolder, F.Cu at (81.5, 59.0)
- added R73: 165 0.1%, Resistor_SMD:R_1206_3216Metric_Pad1.30x1.75mm_HandSolder, F.Cu at (68.7, 37.3)
- added R74: 165 0.1%, Resistor_SMD:R_1206_3216Metric_Pad1.30x1.75mm_HandSolder, F.Cu at (94.2, 52.4)
- added R75: 165 0.1%, Resistor_SMD:R_1206_3216Metric_Pad1.30x1.75mm_HandSolder, F.Cu at (107.0, 52.4)
- added R76: 165 0.1%, Resistor_SMD:R_1206_3216Metric_Pad1.30x1.75mm_HandSolder, F.Cu at (81.5, 30.7)
- added R77: 165 0.1%, Resistor_SMD:R_1206_3216Metric_Pad1.30x1.75mm_HandSolder, F.Cu at (94.2, 30.7)
- added R78: 13K 0.1%, Resistor_SMD:R_1206_3216Metric_Pad1.30x1.75mm_HandSolder, F.Cu at (94.2, 55.7)
- added R79: 1.5K 0.1%, Resistor_SMD:R_1206_3216Metric_Pad1.30x1.75mm_HandSolder, F.Cu at (94.2, 59.0)
- added R80: 13K 0.1%, Resistor_SMD:R_1206_3216Metric_Pad1.30x1.75mm_HandSolder, F.Cu at (107.0, 55.7)
- added R81: 1.5K 0.1%, Resistor_SMD:R_1206_3216Metric_Pad1.30x1.75mm_HandSolder, F.Cu at (107.0, 59.0)
- added R82: 13K 0.1%, Resistor_SMD:R_1206_3216Metric_Pad1.30x1.75mm_HandSolder, F.Cu at (81.5, 34.0)
- added R83: 1.5K 0.1%, Resistor_SMD:R_1206_3216Metric_Pad1.30x1.75mm_HandSolder, F.Cu at (81.5, 37.3)
- added R84: 13K 0.1%, Resistor_SMD:R_1206_3216Metric_Pad1.30x1.75mm_HandSolder, F.Cu at (94.2, 34.0)
- added R85: 1.5K 0.1%, Resistor_SMD:R_1206_3216Metric_Pad1.30x1.75mm_HandSolder, F.Cu at (94.2, 37.3)
- added TP1: TestPoint, TestPoint:TestPoint_Pad_D1.0mm, F.Cu at (75.0, 110.8)
- added TP10: TestPoint, TestPoint:TestPoint_Pad_D1.0mm, F.Cu at (81.5, 88.8)
- added TP11: TestPoint, TestPoint:TestPoint_Pad_D1.0mm, F.Cu at (96.5, 88.8)
- added TP12: TestPoint, TestPoint:TestPoint_Pad_D1.0mm, F.Cu at (111.5, 88.8)
- added TP13: TestPoint, TestPoint:TestPoint_Pad_D1.0mm, F.Cu at (148.2, 135.8)
- added TP14: TestPoint, TestPoint:TestPoint_Pad_D1.0mm, F.Cu at (139.1, 135.8)
- added TP15: TestPoint, TestPoint:TestPoint_Pad_D1.0mm, F.Cu at (126.5, 88.8)
- added TP16: TestPoint, TestPoint:TestPoint_Pad_D1.0mm, F.Cu at (148.2, 149.0)
- added TP2: TestPoint, TestPoint:TestPoint_Pad_D1.0mm, F.Cu at (35.9, 243.9)
- added TP3: TestPoint, TestPoint:TestPoint_Pad_D1.0mm, F.Cu at (40.9, 243.9)
- added TP4: TestPoint, TestPoint:TestPoint_Pad_D1.0mm, F.Cu at (35.9, 235.8)
- added TP5: TestPoint, TestPoint:TestPoint_Pad_D1.0mm, F.Cu at (46.0, 243.9)
- added TP6: TestPoint, TestPoint:TestPoint_Pad_D1.0mm, F.Cu at (51.0, 243.9)
- added TP7: TestPoint, TestPoint:TestPoint_Pad_D1.0mm, F.Cu at (40.9, 235.8)
- added TP8: TestPoint, TestPoint:TestPoint_Pad_D1.0mm, F.Cu at (46.0, 235.8)
- added TP9: TestPoint, TestPoint:TestPoint_Pad_D1.0mm, F.Cu at (66.5, 89.2)
- R10, R15, R5: value 1.5K 0.1% -> 470 0.1%
- R13, R22, R36, R48: value 165 0.1% -> 1.5K 0.1%
- R14, R4, R9: value 13K 0.1% -> 470 0.1%
- R17, R24, R27: value 1k 0.1% -> 910 0.1%
- R18, R30, R42, R8: value 165 0.1% -> 13K 0.1%
- R20, R28, R34, R40: value 13K 0.1% -> 1k 0.1%
- R21, R29, R35, R41: value 1.5K 0.1% -> 1k 0.1%
- R23, R31: value 470 0.1% -> 910 0.1%
- R32: value 1k 0.1% -> 470 0.1%
- moved R3 240.3 mm to (297.1, 73.9)
- moved R60 240.3 mm to (305.2, 48.1)
- moved R61 240.3 mm to (305.2, 51.1)
- moved R62 240.3 mm to (305.2, 54.0)
- moved R63 240.3 mm to (305.2, 57.0)
- moved R64 240.3 mm to (305.2, 60.0)
- moved R65 240.3 mm to (305.2, 62.9)
- moved R66 240.3 mm to (305.2, 65.8)
- moved R67 240.3 mm to (305.2, 68.8)
- moved C21 240.3 mm to (305.3, 45.2)
- moved R9 154.6 mm to (68.7, 20.8)
- moved R40 147.6 mm to (81.5, 27.4)
- moved R41 142.5 mm to (94.2, 27.4)
- moved C18 133.5 mm to (86.9, 20.7)
- moved R8 130.5 mm to (107.0, 24.1)
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Connections:
- net /Analog Channel 1/0-5v/OUTPUT renamed Net-(U3-S3B)
- INPUT1 pad 2: /Analog Channel 1/ADC MUX - TMUX4052/DA -> Net-(D9-COM)
- INPUT2 pad 2: /Analog Channel 5/ADC MUX - TMUX4052/DA -> Net-(D10-COM)
- INPUT3 pad 2: /Analog Channel 2/ADC MUX - TMUX4052/DA -> Net-(D11-COM)
- INPUT4 pad 2: /Analog Channel 3/ADC MUX - TMUX4052/DA -> Net-(D12-COM)
- INPUT5 pad 2: /Analog Channel 4/ADC MUX - TMUX4052/DA -> Net-(D13-COM)
- INPUT6 pad 2: /Analog Channel 6/ADC MUX - TMUX4052/DA -> Net-(D14-COM)
- INPUT7 pad 2: /Analog Channel 7/ADC MUX - TMUX4052/DA -> Net-(D15-COM)
- INPUT8 pad 2: /Analog Channel 8/ADC MUX - TMUX4052/DA -> Net-(D16-COM)
- J1 pad 1: Net-(INPUT1-Pin_1) -> Net-(J1-Pin_1)
- J1 pad 3: Net-(INPUT1-Pin_1) -> Net-(J1-Pin_1)
- J1 pad 5: Net-(INPUT1-Pin_1) -> Net-(J1-Pin_1)
- J2 pad 1: Net-(INPUT2-Pin_1) -> Net-(J2-Pin_1)
- J2 pad 3: Net-(INPUT2-Pin_1) -> Net-(J2-Pin_1)
- J2 pad 5: Net-(INPUT2-Pin_1) -> Net-(J2-Pin_1)
- J3 pad 1: Net-(INPUT3-Pin_1) -> Net-(J3-Pin_1)
- J3 pad 3: Net-(INPUT3-Pin_1) -> Net-(J3-Pin_1)
- J3 pad 5: Net-(INPUT3-Pin_1) -> Net-(J3-Pin_1)
- J4 pad 1: Net-(INPUT4-Pin_1) -> Net-(J4-Pin_1)
- J4 pad 3: Net-(INPUT4-Pin_1) -> Net-(J4-Pin_1)
- J4 pad 5: Net-(INPUT4-Pin_1) -> Net-(J4-Pin_1)
- J5 pad 1: Net-(INPUT5-Pin_1) -> Net-(J5-Pin_1)
- J5 pad 3: Net-(INPUT5-Pin_1) -> Net-(J5-Pin_1)
- J5 pad 5: Net-(INPUT5-Pin_1) -> Net-(J5-Pin_1)
- J6 pad 1: Net-(INPUT6-Pin_1) -> Net-(J6-Pin_1)
- J6 pad 3: Net-(INPUT6-Pin_1) -> Net-(J6-Pin_1)
- J6 pad 5: Net-(INPUT6-Pin_1) -> Net-(J6-Pin_1)
- J7 pad 1: Net-(INPUT7-Pin_1) -> Net-(J7-Pin_1)
- J7 pad 3: Net-(INPUT7-Pin_1) -> Net-(J7-Pin_1)
- J7 pad 5: Net-(INPUT7-Pin_1) -> Net-(J7-Pin_1)
- J8 pad 1: Net-(INPUT8-Pin_1) -> Net-(J8-Pin_1)
- J8 pad 3: Net-(INPUT8-Pin_1) -> Net-(J8-Pin_1)
- J8 pad 5: Net-(INPUT8-Pin_1) -> Net-(J8-Pin_1)
- R1 pad 1: /Analog Channel 1/ADC MUX - TMUX4052/DB -> Net-(U3-DB)
- R10 pad 1: GND -> Net-(U8-S3B)
- R10 pad 2: /Analog Channel 2/0-32v/OUTPUT -> Net-(U8-S3A)
- R11 pad 1: /Analog Channel 2/ADC MUX - TMUX4052/DB -> Net-(U6-DB)
- R13 pad 2: /Analog Channel 2/4-20mA/INPUT -> Net-(U3-S1B)
- R14 pad 1: /Analog Channel 5/0-32v/OUTPUT -> Net-(U10-S3B)
- R14 pad 2: /Analog Channel 5/0-32v/INPUT -> Net-(U10-S3A)
- R15 pad 1: GND -> Net-(U11-S3B)
- R15 pad 2: /Analog Channel 5/0-32v/OUTPUT -> Net-(U11-S3A)
- R17 pad 1: /Analog Channel 1/0-1000 ohm/INPUT -> GND
- R17 pad 2: +3.3V -> Net-(U5-S3B)
- R18 pad 1: GND -> Net-(U5-S1B)
- R18 pad 2: /Analog Channel 5/4-20mA/INPUT -> Net-(U5-S1A)
- R19 pad 1: /Analog Channel 3/ADC MUX - TMUX4052/DB -> Net-(U7-DB)
- R2 pad 2: /Analog Channel 1/0-5v/INPUT -> Net-(U3-S3A)
- R20 pad 1: /Analog Channel 3/0-32v/OUTPUT -> Net-(U3-S2A)
- R20 pad 2: /Analog Channel 3/0-32v/INPUT -> +3.3V
- R21 pad 1: GND -> Net-(U5-S2A)
- R21 pad 2: /Analog Channel 3/0-32v/OUTPUT -> +3.3V
- R22 pad 2: /Analog Channel 3/4-20mA/INPUT -> Net-(U5-S1B)
- R23 pad 1: /Analog Channel 2/0-5v/OUTPUT -> GND
- R23 pad 2: /Analog Channel 2/0-5v/INPUT -> Net-(U6-S3B)
- R24 pad 1: /Analog Channel 2/0-1000 ohm/INPUT -> GND
- R24 pad 2: +3.3V -> Net-(U7-S3B)
- R25 pad 1: /Analog Channel 4/ADC MUX - TMUX4052/DB -> Net-(U8-DB)
- R26 pad 2: /Analog Channel 2/0-5v/OUTPUT -> Net-(U8-S3B)
- R27 pad 1: /Analog Channel 3/0-1000 ohm/INPUT -> GND
- R27 pad 2: +3.3V -> Net-(U10-S3B)
- R28 pad 1: /Analog Channel 4/0-32v/OUTPUT -> Net-(U6-S2A)
- R28 pad 2: /Analog Channel 4/0-32v/INPUT -> +3.3V
- R29 pad 1: GND -> Net-(U7-S2A)
- R29 pad 2: /Analog Channel 4/0-32v/OUTPUT -> +3.3V
- R30 pad 1: GND -> Net-(U6-S1B)
- R30 pad 2: /Analog Channel 4/4-20mA/INPUT -> Net-(U6-S1A)
- R31 pad 1: /Analog Channel 3/0-5v/OUTPUT -> GND
- R31 pad 2: /Analog Channel 3/0-5v/INPUT -> Net-(U11-S3B)
- R32 pad 1: /Analog Channel 4/0-1000 ohm/INPUT -> Net-(U12-S3B)
- R32 pad 2: +3.3V -> Net-(U12-S3A)
- R33 pad 1: /Analog Channel 6/ADC MUX - TMUX4052/DB -> Net-(U10-DB)
- R34 pad 1: /Analog Channel 6/0-32v/OUTPUT -> Net-(U8-S2A)
- R34 pad 2: /Analog Channel 6/0-32v/INPUT -> +3.3V
- R35 pad 1: GND -> Net-(U10-S2A)
- R35 pad 2: /Analog Channel 6/0-32v/OUTPUT -> +3.3V
- R36 pad 2: /Analog Channel 6/4-20mA/INPUT -> Net-(U6-S1B)
- R37 pad 2: /Analog Channel 3/0-5v/OUTPUT -> Net-(U12-S3B)
- R39 pad 1: /Analog Channel 7/ADC MUX - TMUX4052/DB -> Net-(U11-DB)
- R4 pad 1: /Analog Channel 1/0-32v/OUTPUT -> Net-(U5-S3B)
- R4 pad 2: /Analog Channel 1/0-32v/INPUT -> Net-(U5-S3A)
- R40 pad 1: /Analog Channel 7/0-32v/OUTPUT -> Net-(U11-S2A)
- R40 pad 2: /Analog Channel 7/0-32v/INPUT -> +3.3V
- R41 pad 1: GND -> Net-(U12-S2A)
- R41 pad 2: /Analog Channel 7/0-32v/OUTPUT -> +3.3V
- R42 pad 1: GND -> Net-(U7-S1B)
- R42 pad 2: /Analog Channel 7/4-20mA/INPUT -> Net-(U7-S1A)
- R45 pad 1: /Analog Channel 8/ADC MUX - TMUX4052/DB -> Net-(U12-DB)
- R48 pad 2: /Analog Channel 8/4-20mA/INPUT -> Net-(U7-S1B)
- R5 pad 1: GND -> Net-(U6-S3B)
- R5 pad 2: /Analog Channel 1/0-32v/OUTPUT -> Net-(U6-S3A)
- R7 pad 1: /Analog Channel 5/ADC MUX - TMUX4052/DB -> Net-(U5-DB)
- R8 pad 1: GND -> Net-(U3-S1B)
- R8 pad 2: /Analog Channel 1/4-20mA/INPUT -> Net-(U3-S1A)
- R9 pad 1: /Analog Channel 2/0-32v/OUTPUT -> Net-(U7-S3B)
- R9 pad 2: /Analog Channel 2/0-32v/INPUT -> Net-(U7-S3A)
- U1 pad 12: unconnected-(U1-GPIO8-Pad12) -> SDA
- U1 pad 15: unconnected-(U1-GPIO9-Pad15) -> SCL
- U1 pad 21: unconnected-(U1-5V0-Pad21) -> +5V
- U2 pad 1: +3.3V -> GND
- U9 pad 1: unconnected-(U9-SW-Pad1) -> Net-(D17-A)
- U9 pad 2: unconnected-(U9-GND-Pad2) -> GND
- U9 pad 3: unconnected-(U9-FB-Pad3) -> Net-(U9-FB)
- U9 pad 4: unconnected-(U9-EN-Pad4) -> +5V
- U9 pad 5: unconnected-(U9-VIN-Pad5) -> +5V

Commit message: changed from mux to pin jumpers
Parts:
- removed C10, C12, C14, C16, C18, C20, C5, C9: 100nF, Capacitor_SMD:C_0805_2012Metric_Pad1.18x1.45mm_HandSolder
- removed D10, D11, D12, D13, D14, D15, D16, D9: BAV199, Package_TO_SOT_SMD:SOT-23
- removed R3: 10K, Resistor_SMD:R_1206_3216Metric_Pad1.30x1.75mm_HandSolder
- removed TP1, TP10, TP11, TP12, TP13, TP14, TP15, TP16, TP2, TP3, TP4, TP5, TP6, TP7, TP8, TP9: TestPoint, TestPoint:TestPoint_Pad_D1.0mm
- added H10: MountingHole_Pad, MountingHole:MountingHole_3.2mm_M3_ISO14580_Pad, F.Cu at (66.0, 62.0)
- added H11: MountingHole_Pad, MountingHole:MountingHole_3.2mm_M3_ISO14580_Pad, F.Cu at (229.0, 62.0)
- added H12: MountingHole_Pad, MountingHole:MountingHole_3.2mm_M3_ISO14580_Pad, F.Cu at (229.0, 123.0)
- added H13: MountingHole_Pad, MountingHole:MountingHole_3.2mm_M3_ISO14580_Pad, F.Cu at (66.0, 123.0)
- added J10: Conn_02x05_Odd_Even, Connector_PinHeader_2.54mm:PinHeader_2x05_P2.54mm_Vertical_SMD, F.Cu at (121.0, 94.0)
- added J11: Conn_02x05_Odd_Even, Connector_PinHeader_2.54mm:PinHeader_2x05_P2.54mm_Vertical_SMD, F.Cu at (135.0, 96.5)
- added J12: Conn_02x05_Odd_Even, Connector_PinHeader_2.54mm:PinHeader_2x05_P2.54mm_Vertical_SMD, F.Cu at (149.0, 96.5)
- added J13: Conn_02x05_Odd_Even, Connector_PinHeader_2.54mm:PinHeader_2x05_P2.54mm_Vertical_SMD, F.Cu at (163.0, 96.5)
- added J14: Conn_02x05_Odd_Even, Connector_PinHeader_2.54mm:PinHeader_2x05_P2.54mm_Vertical_SMD, F.Cu at (191.0, 96.5)
- added J15: Conn_02x05_Odd_Even, Connector_PinHeader_2.54mm:PinHeader_2x05_P2.54mm_Vertical_SMD, F.Cu at (205.0, 96.5)
- added J16: Conn_02x05_Odd_Even, Connector_PinHeader_2.54mm:PinHeader_2x05_P2.54mm_Vertical_SMD, F.Cu at (177.0, 96.5)
- added J17: Conn_02x05_Odd_Even, Connector_PinHeader_2.54mm:PinHeader_2x05_P2.54mm_Vertical_SMD, F.Cu at (219.0, 96.5)
- added J18: Conn_02x05_Odd_Even, Connector_PinHeader_2.54mm:PinHeader_2x05_P2.54mm_Vertical_SMD, F.Cu at (121.0, 72.0)
- added J19: Conn_02x05_Odd_Even, Connector_PinHeader_2.54mm:PinHeader_2x05_P2.54mm_Vertical_SMD, F.Cu at (135.0, 77.5)
- added J20: Conn_02x05_Odd_Even, Connector_PinHeader_2.54mm:PinHeader_2x05_P2.54mm_Vertical_SMD, F.Cu at (149.0, 77.5)
- added J21: Conn_02x05_Odd_Even, Connector_PinHeader_2.54mm:PinHeader_2x05_P2.54mm_Vertical_SMD, F.Cu at (163.0, 77.5)
- added J22: Conn_02x05_Odd_Even, Connector_PinHeader_2.54mm:PinHeader_2x05_P2.54mm_Vertical_SMD, F.Cu at (191.0, 77.5)
- added J23: Conn_02x05_Odd_Even, Connector_PinHeader_2.54mm:PinHeader_2x05_P2.54mm_Vertical_SMD, F.Cu at (205.0, 77.5)
- added J24: Conn_02x05_Odd_Even, Connector_PinHeader_2.54mm:PinHeader_2x05_P2.54mm_Vertical_SMD, F.Cu at (177.0, 77.5)
- added J25: Conn_02x05_Odd_Even, Connector_PinHeader_2.54mm:PinHeader_2x05_P2.54mm_Vertical_SMD, F.Cu at (219.0, 77.5)
- added R38: 10k 0.1%, Resistor_SMD:R_0603_1608Metric, F.Cu at (123.5, 86.0)
- added R43: 10k 0.1%, Resistor_SMD:R_0603_1608Metric, F.Cu at (137.5, 88.5)
- added R44: 10k 0.1%, Resistor_SMD:R_0603_1608Metric, F.Cu at (151.5, 88.5)
- added R46: 10k 0.1%, Resistor_SMD:R_0603_1608Metric, F.Cu at (165.5, 88.5)
- added R47: 10k 0.1%, Resistor_SMD:R_0603_1608Metric, F.Cu at (193.5, 88.5)
- added R49: 10k 0.1%, Resistor_SMD:R_0603_1608Metric, F.Cu at (207.5, 88.5)
- added R50: 10k 0.1%, Resistor_SMD:R_0603_1608Metric, F.Cu at (179.5, 88.5)
- added R51: 10k 0.1%, Resistor_SMD:R_0603_1608Metric, F.Cu at (221.5, 88.5)
- added TP81: TestPoint, TestPoint:TestPoint_Pad_D1.0mm, F.Cu at (126.0, 64.0)
- added TP82: TestPoint, TestPoint:TestPoint_Pad_D1.0mm, F.Cu at (140.0, 70.0)
- added TP83: TestPoint, TestPoint:TestPoint_Pad_D1.0mm, F.Cu at (154.0, 70.0)
- added TP84: TestPoint, TestPoint:TestPoint_Pad_D1.0mm, F.Cu at (168.0, 70.0)
- added TP85: TestPoint, TestPoint:TestPoint_Pad_D1.0mm, F.Cu at (196.0, 70.0)
- added TP86: TestPoint, TestPoint:TestPoint_Pad_D1.0mm, F.Cu at (210.0, 70.0)
- added TP87: TestPoint, TestPoint:TestPoint_Pad_D1.0mm, F.Cu at (182.0, 70.0)
- added TP88: TestPoint, TestPoint:TestPoint_Pad_D1.0mm, F.Cu at (224.0, 70.0)
- added TP89: TestPoint, TestPoint:TestPoint_Pad_D1.0mm, F.Cu at (121.0, 113.5)
- added TP90: TestPoint, TestPoint:TestPoint_Pad_D1.0mm, F.Cu at (140.5, 113.5)
- added TP91: TestPoint, TestPoint:TestPoint_Pad_D1.0mm, F.Cu at (154.5, 113.5)
- added TP92: TestPoint, TestPoint:TestPoint_Pad_D1.0mm, F.Cu at (168.5, 113.5)
- added TP93: TestPoint, TestPoint:TestPoint_Pad_D1.0mm, F.Cu at (196.5, 113.5)
- added TP94: TestPoint, TestPoint:TestPoint_Pad_D1.0mm, F.Cu at (210.5, 113.5)
- added TP95: TestPoint, TestPoint:TestPoint_Pad_D1.0mm, F.Cu at (182.5, 113.5)
- added TP96: TestPoint, TestPoint:TestPoint_Pad_D1.0mm, F.Cu at (224.5, 113.5)
- J1, J2, J3, J4, J5, J6, J7, J8: footprint Connector_PinHeader_2.54mm:PinHeader_2x03_P2.54mm_Vertical -> Connector_PinHeader_2.54mm:PinHeader_2x03_P2.54mm_Vertical_SMD
- R10, R13, R14, R15, R16, R17, R18, R2, R20, R21, R22, R23, R24, R26, R27, R28, R29, R30, R31, R32, R34, R35, R36, R37, R4, R40, R41, R42, R48, R5, R78, R79, R8, R80, R81, R82, R83, R84, R85, R9: footprint Resistor_SMD:R_1206_3216Metric_Pad1.30x1.75mm_HandSolder -> Resistor_SMD:R_0603_1608Metric
- moved R63 238.1 mm to (72.2, 106.0), turned to 90 degrees
- moved R62 235.2 mm to (75.0, 102.0), turned to 90 degrees
- moved R64 234.7 mm to (75.2, 106.0), turned to 90 degrees
- moved C21 234.2 mm to (78.1, 102.0), turned to 90 degrees
- moved R65 231.2 mm to (78.1, 106.0), turned to 90 degrees
- moved R60 230.6 mm to (81.0, 102.0), turned to 90 degrees
- moved R66 227.8 mm to (81.0, 106.0), turned to 90 degrees
- moved R61 227.0 mm to (84.0, 102.0), turned to 90 degrees
- moved R67 224.4 mm to (84.0, 106.0), turned to 90 degrees
- moved C7 156.7 mm to (74.2, 82.5)
- moved C8 156.7 mm to (74.2, 85.5)
- moved R12 156.7 mm to (79.0, 82.5)
- moved U4 156.7 mm to (75.3, 78.7)
- moved U9 155.5 mm to (79.0, 96.6), turned to 90 degrees
- moved C2 148.3 mm to (74.2, 69.9)
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Routing:
- net Net-(INPUT1-Pin_2): track 0.00 -> 30.7 mm
- net Net-(J10-Pin_6): track 0.00 -> 17.8 mm
- net Net-(J10-Pin_8): track 0.00 -> 17.6 mm
- net Net-(J18-Pin_10): track 0.00 -> 15.2 mm
- net Net-(J18-Pin_3): track 0.00 -> 11.3 mm
- net Net-(J18-Pin_9): track 0.00 -> 11.3 mm
- net /ADC1/ADC0: track 0.00 -> 11.1 mm
- net Net-(J1-Pin_1): track 0.00 -> 9.48 mm
- net Net-(J10-Pin_2): track 0.00 -> 5.46 mm
- net Net-(J10-Pin_10): track 0.00 -> 4.68 mm
- net Net-(J10-Pin_4): track 0.00 -> 4.67 mm
- net Net-(INPUT1-Pin_1): track 0.00 -> 4.16 mm
Other:
- board outline added: 169 x 67 mm

Commit message: layout work.
Parts:
- added C10: 10uF, Capacitor_SMD:C_0603_1608Metric, F.Cu at (109.8, 92.8)
- added C11: 22pF, Capacitor_SMD:C_0603_1608Metric, F.Cu at (101.8, 95.8)
- added C12: 1uF, Capacitor_SMD:C_1206_3216Metric, F.Cu at (101.5, 90.5)
- added L1: 10uH, Inductor_SMD:L_Ferrocore_DLG-0403, F.Cu at (107.2, 86.8)
- added R43: 1.87M, Resistor_SMD:R_0603_1608Metric, F.Cu at (101.8, 93.8)
- added R44: 100k, Resistor_SMD:R_0603_1608Metric, F.Cu at (106.0, 95.8)
- moved U2 33.0 mm to (108.2, 67.5)
- moved U3 33.0 mm to (108.2, 77.2)
- moved R71 31.7 mm to (106.5, 105.8)
- moved R69 31.7 mm to (112.5, 105.8)
- moved R74 30.4 mm to (108.5, 105.8)
- moved R72 30.3 mm to (102.5, 105.8)
- moved C6 30.2 mm to (104.0, 77.3), turned to -90 degrees
- moved C2 29.8 mm to (104.0, 67.5), turned to -90 degrees
- moved R75 29.4 mm to (104.5, 105.8)
- moved C7 28.7 mm to (101.8, 77.3), turned to -90 degrees
- moved J25 28.5 mm to (105.5, 117.0)
- moved D6 28.4 mm to (101.8, 86.8), turned to 0 degrees
- moved C3 28.0 mm to (101.8, 67.5), turned to -90 degrees
- moved C16 27.8 mm to (105.8, 99.8), turned to 0 degrees
- moved U4 27.7 mm to (106.5, 93.0), turned to 0 degrees
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- renumbered C15 to C13, C17 to C14, C19 to C15, C21 to C16, C6 to C5, C7 to C6, C8 to C7, C11 to C8, C13 to C9, D17 to D6, D6 to D7, D7 to D8, D8 to D9, H10 to H1, H11 to H2, H12 to H3, H13 to H4, J4 to J10, J13 to J11, J21 to J12, J5 to J13, J22 to J15, J6 to J16, J15 to J17, J23 to J18, J7 to J19, J10 to J2, J16 to J20, J24 to J21, J8 to J22, J17 to J23, J25 to J24, J9 to J25, J18 to J3, J2 to J4, J11 to J5, J19 to J6, J3 to J7, J12 to J8, J20 to J9, R70 to R1, R71 to R10, R18 to R11, R22 to R12, R21 to R13, R43 to R14, R4 to R15, R17 to R16, R7 to R17, R72 to R18, R30 to R19, R8 to R2, R36 to R20, R28 to R21, R44 to R22, R5 to R23, R23 to R24, R11 to R25, R12 to R26, R73 to R27, R42 to R28, R48 to R29, R13 to R3, R29 to R30, R46 to R31, R9 to R32, R24 to R33, R19 to R34, R74 to R35, R78 to R36, R79 to R37, R34 to R38, R47 to R39, R20 to R4, R10 to R40, R26 to R41, R25 to R42, R75 to R45, R80 to R46, R81 to R47, R35 to R48, R38 to R5, R14 to R50, R27 to R51, R33 to R52, R76 to R53, R82 to R54, R83 to R55, R40 to R56, R50 to R57, R15 to R58, R31 to R59, R2 to R6, R39 to R60, R77 to R61, R84 to R62, R85 to R63, R41 to R64, R51 to R65, R32 to R66, R37 to R67, R45 to R68, R60 to R69, R16 to R7, R61 to R70, R62 to R71, R63 to R72, R67 to R73, R65 to R74, R64 to R75, R66 to R76, R1 to R8, R6 to R9, TP89 to TP1, TP85 to TP10, TP94 to TP11, TP86 to TP12, TP95 to TP13, TP87 to TP14, TP96 to TP15, TP88 to TP16, TP81 to TP2, TP90 to TP3, TP82 to TP4, TP91 to TP5, TP83 to TP6, TP92 to TP7, TP84 to TP8, TP93 to TP9, U4 to U3, U9 to U4
Routing:
- net Net-(INPUT1-Pin_2): track 30.7 -> 0.00 mm
- net Net-(J2-Pin_6): track 17.8 -> 0.00 mm
- net Net-(J2-Pin_8): track 17.6 -> 0.00 mm
- net Net-(J3-Pin_10): track 15.2 -> 0.00 mm
- net Net-(J3-Pin_3): track 11.3 -> 0.00 mm
- net Net-(J3-Pin_9): track 11.3 -> 0.00 mm
- net /ADC1/ADC0: track 11.1 -> 0.00 mm
- net Net-(J1-Pin_1): track 9.48 -> 0.00 mm
- net Net-(J2-Pin_2): track 5.46 -> 0.00 mm
- net Net-(J2-Pin_10): track 4.68 -> 0.00 mm
- net Net-(J2-Pin_4): track 4.67 -> 0.00 mm
- net Net-(INPUT8-Pin_1): track 0.00 -> 4.61 mm
- net Net-(INPUT7-Pin_1): track 0.00 -> 4.61 mm
- net Net-(INPUT6-Pin_1): track 0.00 -> 4.61 mm
- net Net-(INPUT5-Pin_1): track 0.00 -> 4.61 mm
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Other:
- board size 169 x 67 mm -> 169 x 63.5 mm
- board text added: "10kΩ"
- board text added: "1kΩ"
- board text added: "32v"
- board text added: "420"
- board text added: "5v"
