File: sendit/adc.kicad_sch (KiCad schematic)
At the start: 17 parts, among them U6 MCP3564R

Commit message: brought over the latest esp32-s3 schematic
Parts:
- renumbered R18 to R19, R19 to R20, R20 to R21, R21 to R22, R22 to R23, R23 to R24, R24 to R25, R25 to R26, R26 to R27
Changed lines of the file:
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@@
 		(on_board yes)
 		(dnp no)
-		(property "Reference" "R24"
+		(property "Reference" "R25"
 			(at 172.974 108.204 90)
 			(effects
@@
 			(project "sendit"
 				(path "/a355e4d0-2918-44fc-be8d-2503b84c6d6c/012ce78d-7e37-48fe-89b4-0e95092577e6"
-					(reference "R24")
+					(reference "R25")
 					(unit 1)
 				)
@@
 		(on_board yes)
 		(dnp no)
-		(property "Reference" "R21"
+		(property "Reference" "R22"
 			(at 164.084 105.664 90)
 			(effects
@@
 			(project "sendit"
 				(path "/a355e4d0-2918-44fc-be8d-2503b84c6d6c/012ce78d-7e37-48fe-89b4-0e95092577e6"
-					(reference "R21")
+					(reference "R22")
 					(unit 1)
 				)
@@
 		(on_board yes)
 		(dnp no)
-		(property "Reference" "R18"
+		(property "Reference" "R19"
 			(at 141.224 75.946 90)
 			(effects
@@
 			(project "sendit"
 				(path "/a355e4d0-2918-44fc-be8d-2503b84c6d6c/012ce78d-7e37-48fe-89b4-0e95092577e6"
-					(reference "R18")
+					(reference "R19")
 					(unit 1)
 				)
@@
 		(on_board yes)
 		(dnp no)
-		(property "Reference" "R22"
+		(property "Reference" "R23"
 			(at 164.084 110.744 90)
 			(effects
@@
 			(project "sendit"
 				(path "/a355e4d0-2918-44fc-be8d-2503b84c6d6c/012ce78d-7e37-48fe-89b4-0e95092577e6"
-					(reference "R22")
+					(reference "R23")
 					(unit 1)
 				)
@@
 		(on_board yes)
 		(dnp no)
-		(property "Reference" "R20"
+		(property "Reference" "R21"
 			(at 164.084 95.504 90)
 			(effects
@@
 			(project "sendit"
 				(path "/a355e4d0-2918-44fc-be8d-2503b84c6d6c/012ce78d-7e37-48fe-89b4-0e95092577e6"
-					(reference "R20")
+					(reference "R21")
 					(unit 1)
 				)
@@
 		(on_board yes)
 		(dnp no)
-		(property "Reference" "R19"
+		(property "Reference" "R20"
 			(at 148.844 75.946 90)
 			(effects
@@
 			(project "sendit"
 				(path "/a355e4d0-2918-44fc-be8d-2503b84c6d6c/012ce78d-7e37-48fe-89b4-0e95092577e6"
-					(reference "R19")
+					(reference "R20")
 					(unit 1)
 				)
@@
 		(on_board yes)
 		(dnp no)
-		(property "Reference" "R25"
+		(property "Reference" "R26"
 			(at 172.974 113.284 90)
 			(effects
@@
 			(project "sendit"
 				(path "/a355e4d0-2918-44fc-be8d-2503b84c6d6c/012ce78d-7e37-48fe-89b4-0e95092577e6"
-					(reference "R25")
+					(reference "R26")
 					(unit 1)
 				)
@@
 		(on_board yes)
 		(dnp yes)
-		(property "Reference" "R23"
+		(property "Reference" "R24"
 			(at 172.974 98.044 90)
 			(effects
@@
 			(project "sendit"
 				(path "/a355e4d0-2918-44fc-be8d-2503b84c6d6c/012ce78d-7e37-48fe-89b4-0e95092577e6"
-					(reference "R23")
+					(reference "R24")
 					(unit 1)
 				)
@@
 		(dnp no)
 		(fields_autoplaced yes)
-		(property "Reference" "R26"
+		(property "Reference" "R27"
 			(at 180.34 86.3599 0)
 			(effects
@@
 			(project "sendit"
 				(path "/a355e4d0-2918-44fc-be8d-2503b84c6d6c/012ce78d-7e37-48fe-89b4-0e95092577e6"
-					(reference "R26")
-					(unit 1)
-				)
+					(reference "R27")
+					(unit 1)
+				)

Commit message: passing erc and drc
Changed lines of the file:
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@@
+	)
+	(symbol
+		(lib_id "power:PWR_FLAG")
+		(at 156.21 78.74 0)
+		(unit 1)
+		(exclude_from_sim no)
+		(in_bom yes)
+		(on_board yes)
+		(dnp no)
+		(property "Reference" "#FLG08"
+			(at 156.21 76.835 0)
+			(effects
+				(font
+					(size 1.27 1.27)
+				)
+				(hide yes)
+			)
+		)
+		(property "Value" "PWR_FLAG"
+			(at 156.21 74.93 0)
+			(effects
+				(font
+					(size 1.27 1.27)
+				)
+			)
+		)
+		(property "Footprint" ""
+			(at 156.21 78.74 0)
+			(effects
+				(font
+					(size 1.27 1.27)
+				)
+				(hide yes)
+			)
+		)
+		(property "Datasheet" "~"
+			(at 156.21 78.74 0)
+			(effects
+				(font
+					(size 1.27 1.27)
+				)
+				(hide yes)
+			)
+		)
+		(property "Description" "Special symbol for telling ERC where power comes from"
+			(at 156.21 78.74 0)
+			(effects
+				(font
+					(size 1.27 1.27)
+				)
+				(hide yes)
+			)
+		)
+		(pin "1"
+		)
+		(instances
+			(project "sendit"
+				(path "/a355e4d0-2918-44fc-be8d-2503b84c6d6c/012ce78d-7e37-48fe-89b4-0e95092577e6"
+					(reference "#FLG08")
+					(unit 1)
+				)
+			)
+		)
 	)
 	(symbol
@@
 					(unit 1)
 				)
+			)
+		)
+	)
+	(symbol
+		(lib_id "power:PWR_FLAG")
+		(at 129.54 78.74 0)
+		(unit 1)
+		(exclude_from_sim no)
+		(in_bom yes)
+		(on_board yes)
+		(dnp no)
+		(property "Reference" "#FLG07"
+			(at 129.54 76.835 0)
+			(effects
+				(font
+					(size 1.27 1.27)
+				)
+				(hide yes)
+			)
+		)
+		(property "Value" "PWR_FLAG"
+			(at 129.54 74.93 0)
+			(effects
+				(font
+					(size 1.27 1.27)
+				)
+			)
+		)
+		(property "Footprint" ""
+			(at 129.54 78.74 0)
+			(effects
+				(font
+					(size 1.27 1.27)
+				)
+				(hide yes)
+			)
+		)
+		(property "Datasheet" "~"
+			(at 129.54 78.74 0)
+			(effects
+				(font
+					(size 1.27 1.27)
+				)
+				(hide yes)
+			)
+		)
+		(property "Description" "Special symbol for telling ERC where power comes from"
+			(at 129.54 78.74 0)
+			(effects
+				(font
+					(size 1.27 1.27)
+				)
+				(hide yes)
+			)
+		)
+		(pin "1"
+		)
+		(instances
+			(project "sendit"
+				(path "/a355e4d0-2918-44fc-be8d-2503b84c6d6c/012ce78d-7e37-48fe-89b4-0e95092577e6"
+					(reference "#FLG07")
+					(unit 1)
+				)

Commit message: cleaning up schematics a bit for design review
Other:
- title: FrothFET 8CH -> https://github.com/hoeken/sendit
Changed lines of the file:
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@@
 	(paper "A4")
 	(title_block
-		(title "FrothFET 8CH")
-		(date "2024-08-21")
-		(rev "E")
+		(title "https://github.com/hoeken/sendit")
+		(date "2025-08-28")
+		(rev "B")
 		(company "https://github.com/hoeken/frothfet")
 	)
